File: Blank_Project_2.kicad_sch (KiCad schematic)
At the start: 8 parts

Commit message: Update Blank_Project_2.kicad_sch
Line 249 changed "R1" to "R1 change in GitHub"
Parts:
- R1 change in GitHub: renamed from R1
Changed lines of the file:
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@@
   (symbol (lib_id "Device:R") (at 73.66 87.63 0) (unit 1)
     (in_bom yes) (on_board yes) (dnp no) (fields_autoplaced)
-    (property "Reference" "R1" (at 76.2 86.36 0)
+    (property "Reference" "R1 change in GitHub" (at 76.2 86.36 0)
       (effects (font (size 1.27 1.27)) (justify left))
     )
